File: fieldeffect4.sch (KiCad schematic (older format))
At the start: 20 parts

Commit message: add netlist
Parts:
- added J1, J2, J3, J4, J5: Conn_01x02, Sockets_MOLEX_KK-System:Socket_MOLEX-KK-RM3-96mm_Lock_2pin_straight, symbol Connector_Generic:Conn_01x02
- added J10, J6, J7, J8, J9: Conn_01x02, Connector_PinHeader_2.54mm:PinHeader_1x02_P2.54mm_Vertical, symbol Connector_Generic:Conn_01x02
- C1, C2, C3, C4, C5, C6, C7, C8: renamed from C?; footprint (none) -> Capacitor_SMD:C_0603_1608Metric
- D1, D2, D3, D4: renamed from D?; footprint (none) -> Capacitor_SMD:C_0603_1608Metric
- Q1, Q2, Q3, Q4: renamed from Q?; footprint (none) -> Package_TO_SOT_SMD:TO-263-2
- gave numbers to parts that had none: 4
Connections:
- net labels added: +48V
- wire segments 60 -> 105
