File: fieldeffector.kicad_pcb (KiCad board)
At the start: 2 copper layers, 30 parts, among them J1 Conn_01x02, J10 Conn_01x02, J2 Conn_01x02, J3 Conn_01x02, J4 Conn_01x02, J5 Conn_01x02, J6 Conn_01x02, J7 Conn_01x02, J8 Conn_01x02, J9 Conn_01x02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

Commit message: update layout
Parts:
- added H1: MountingHole, MountingHole:MountingHole_3.2mm_M3, F.Cu at (73.4, 128.1)
- added H2: MountingHole, MountingHole:MountingHole_3.2mm_M3, F.Cu at (153.7, 88.1)
- added H3: MountingHole, MountingHole:MountingHole_3.2mm_M3, F.Cu at (153.7, 128.1)
- added H4: MountingHole, MountingHole:MountingHole_3.2mm_M3, F.Cu at (73.4, 88.1)
- moved J6 6.79 mm to (82.9, 126.9)
- moved C5 6.73 mm to (121.7, 127.8), turned to 180 degrees
- moved C7 6.71 mm to (137.9, 127.8), turned to 180 degrees
- moved C4 6.66 mm to (105.4, 127.8), turned to 180 degrees
- moved C2 6.62 mm to (89.1, 127.8), turned to 180 degrees
- moved C1 0.29 mm to (89.2, 125.8)
- moved C6 0.28 mm to (121.7, 125.8)
- moved C3 0.26 mm to (105.4, 125.8)
- moved C8 0.21 mm to (137.9, 125.8)
Routing:
- net +5V: track 0.00 -> 26.3 mm, vias 0 -> 4
Other:
- board outline added: 88.2 x 48 mm
